Commit message: Edited gazebo xacro files to include grasping plugin

File: xarm_description/urdf/common/common.gazebo.xacro (robot description, xacro)
@@ -1,4 +1,5 @@
 <?xml version="1.0"?>
 <robot xmlns:xacro="http://ros.org/wiki/xacro">
+  <!-- ROS2 Control Plugin for Ignition -->
   <xacro:macro name="ignition_ros2_control_plugin" params="prefix:='' ros2_control_params:=''">
     <gazebo>
@@ -7,8 +8,10 @@
           <parameters>${ros2_control_params}</parameters>
         </xacro:if>
+        <!-- Optionally specify a controller manager node name -->
         <!-- <controller_manager_node_name>${prefix}controller_manager</controller_manager_node_name> -->
       </plugin>
     </gazebo>
   </xacro:macro>
+  <!-- ROS2 Control Plugin -->
   <xacro:macro name="gazebo_ros2_control_plugin" params="ros2_control_params:=''">
     <gazebo>
@@ -21,4 +24,5 @@
     </gazebo>
   </xacro:macro>
+  <!-- ROS1 Control Plugin -->
   <xacro:macro name="gazebo_ros1_control_plugin" params="namespace:=''">
     <gazebo>
@@ -27,8 +31,43 @@
         <!-- <controlPeriod>0.0001</controlPeriod> -->
         <robotSimType>gazebo_ros_control/DefaultRobotHWSim</robotSimType>
-		    <legacyModeNS>true</legacyModeNS>
+        <legacyModeNS>true</legacyModeNS>
         <!-- <preserveWorldVelocity>true</preserveWorldVelocity> -->
       </plugin>
     </gazebo>
   </xacro:macro>
+  <!-- Grasp Fix Plugin Macro -->
+  <xacro:macro name="gazebo_grasp_fix_plugin" params="arm_name:='', palm_link1:='', palm_link2:='', gripper_link1:='', gripper_link2:=''">
+    <gazebo>
+      <plugin name="gazebo_grasp_fix" filename="libgazebo_grasp_fix.so">
+        <arm>
+          <arm_name>${arm_name}</arm_name>
+          <palm_link>${palm_link1}</palm_link>
+          <palm_link>${palm_link2}</palm_link>
+          <gripper_link>${gripper_link1}</gripper_link>
+          <gripper_link>${gripper_link2}</gripper_link>
+        </arm>
+        <forces_angle_tolerance>100</forces_angle_tolerance>
+        <update_rate>4</update_rate>
+        <grip_count_threshold>4</grip_count_threshold>
+        <max_grip_count>8</max_grip_count>
+        <release_tolerance>0.005</release_tolerance>
+        <disable_collisions_on_attach>false</disable_collisions_on_attach>
+        <contact_topic>__default_topic__</contact_topic>
+      </plugin>
+    </gazebo>
+  </xacro:macro>
+  <!-- Composite Macro: Loads one control plugin (based on a parameter) and then the grasp fix plugin -->
+  <xacro:macro name="gazebo_plugins" params="ros2_control_params:='', prefix:='', control_plugin_type:='ros2', arm_name:='', palm_link1:='', palm_link2:='' gripper_link1:='', gripper_link2:=''">
+    <xacro:if value="${control_plugin_type == 'ignition'}">
+      <xacro:ignition_ros2_control_plugin prefix="${prefix}" ros2_control_params="${ros2_control_params}"/>
+    </xacro:if>
+    <xacro:if value="${control_plugin_type == 'ros2'}">
+      <xacro:gazebo_ros2_control_plugin ros2_control_params="${ros2_control_params}"/>
+    </xacro:if>
+    <xacro:if value="${control_plugin_type == 'ros1'}">
+      <xacro:gazebo_ros1_control_plugin namespace="${prefix}"/>
+    </xacro:if>
+    <!-- Load the grasp fix plugin -->
+    <xacro:gazebo_grasp_fix_plugin arm_name="${arm_name}" palm_link1="${palm_link1}" palm_link2="${palm_link2}" gripper_link1="${gripper_link1}" gripper_link2="${gripper_link2}"/>
+  </xacro:macro>
 </robot>

File: xarm_description/urdf/xarm_device_macro.xacro (robot description, xacro)
@@ -42,6 +42,5 @@
     mesh_suffix:='stl'
     kinematics_suffix:=''
-    "
-    >
+    ">
     <!-- Load Common Material -->
     <xacro:include filename="$(find xarm_description)/urdf/_private_macro.xacro" />
@@ -202,5 +201,5 @@
     </xacro:unless>
     <xacro:if value="${add_realsense_d435i}">
-      <!-- (xarm) Load RealSense D435i URDF -->
+      <!-- Load RealSense D435i URDF -->
       <xacro:include filename="$(find xarm_description)/urdf/camera/realsense_d435i.urdf.xacro" />
       <xacro:d435i_urdf prefix="${prefix}" add_d435i_links="${add_d435i_links}" />
@@ -251,19 +250,9 @@
       </xacro:unless>
     </xacro:if>
-    <xacro:if value="${not add_gripper and not add_vacuum_gripper and add_other_geometry}">
-      <!-- Load Other Model URDF -->
-      <xacro:include filename="$(find xarm_description)/urdf/other/other_geometry.urdf.xacro" />
-      <xacro:other_geometry prefix="${prefix}" attach_to="${prefix}link_eef"
-        geometry_type="${geometry_type}" geometry_mass="${geometry_mass}"
-        geometry_height="${geometry_height}" geometry_radius="${geometry_radius}"
-        geometry_length="${geometry_length}" geometry_width="${geometry_width}"
-        geometry_mesh_filename="${geometry_mesh_filename}"
-        geometry_mesh_origin_xyz="${geometry_mesh_origin_xyz}" geometry_mesh_origin_rpy="${geometry_mesh_origin_rpy}"
-        geometry_mesh_tcp_xyz="${geometry_mesh_tcp_xyz}" geometry_mesh_tcp_rpy="${geometry_mesh_tcp_rpy}"
-      />
-    </xacro:if>
-    <!-- gazebo_plugin -->
+    <!-- gazebo_plugin block -->
     <xacro:if value="${load_gazebo_plugin}">
+      <!-- Include common gazebo macros -->
       <xacro:include filename="$(find xarm_description)/urdf/common/common.gazebo.xacro" />
+      <!-- Define new_ros2_control_params if in ROS2 -->
       <xacro:if value="${is_ros2}">
         <xacro:if value="${robot_type == 'uf850' or robot_type == 'xarm7_mirror'}">
@@ -276,14 +265,15 @@
           <xacro:property name="new_ros2_control_params" value="${ros2_control_params}"/>
         </xacro:if>
-        <xacro:if value="${ros2_control_plugin == 'ign_ros2_control/IgnitionSystem'}">
-          <xacro:ignition_ros2_control_plugin prefix="${prefix}" ros2_control_params="${new_ros2_control_params}"/>
-        </xacro:if>
-        <xacro:unless value="${ros2_control_plugin == 'ign_ros2_control/IgnitionSystem'}">
-          <xacro:gazebo_ros2_control_plugin ros2_control_params="${new_ros2_control_params}"/>
-        </xacro:unless>
-      </xacro:if>
-      <xacro:unless value="${is_ros2}">
-        <xacro:gazebo_ros1_control_plugin namespace="${hw_ns}"/>
-      </xacro:unless>
+      </xacro:if>
+      <!-- Use composite macro to load control plugin and grasp fix plugin once -->
+      <xacro:gazebo_plugins
+        ros2_control_params="${new_ros2_control_params}"
+        prefix="${prefix}"
+        control_plugin_type="ros2"
+        arm_name="xarm7"
+        palm_link1="left_inner_knuckle"
+        palm_link2="right_inner_knuckle"
+        gripper_link1="left_finger"
+        gripper_link2="right_finger"/>
     </xacro:if>
     <xacro:if value="${use_gazebo_camera}">

Commit message: Pick and place working in sim somewhat consistently

File: xarm_description/urdf/common/common.gazebo.xacro (robot description, xacro)
@@ -47,9 +47,9 @@
           <gripper_link>${gripper_link2}</gripper_link>
         </arm>
-        <forces_angle_tolerance>100</forces_angle_tolerance>
-        <update_rate>4</update_rate>
-        <grip_count_threshold>4</grip_count_threshold>
-        <max_grip_count>8</max_grip_count>
-        <release_tolerance>0.005</release_tolerance>
+        <forces_angle_tolerance>160</forces_angle_tolerance>
+        <update_rate>20</update_rate>
+        <grip_count_threshold>2</grip_count_threshold>
+        <max_grip_count>12</max_grip_count>
+        <release_tolerance>0.01</release_tolerance>
         <disable_collisions_on_attach>false</disable_collisions_on_attach>
         <contact_topic>__default_topic__</contact_topic>
@@ -58,5 +58,5 @@
   </xacro:macro>
   <!-- Composite Macro: Loads one control plugin (based on a parameter) and then the grasp fix plugin -->
-  <xacro:macro name="gazebo_plugins" params="ros2_control_params:='', prefix:='', control_plugin_type:='ros2', arm_name:='', palm_link1:='', palm_link2:='' gripper_link1:='', gripper_link2:=''">
+  <xacro:macro name="gazebo_plugins" params="ros2_control_params:='', prefix:='', control_plugin_type:='ros2', arm_name:='', palm_link1:='', palm_link2:='', gripper_link1:='', gripper_link2:=''">
     <xacro:if value="${control_plugin_type == 'ignition'}">
       <xacro:ignition_ros2_control_plugin prefix="${prefix}" ros2_control_params="${ros2_control_params}"/>
