Commit message: Added working FT_sensor URDF to xarm7

File: xarm_description/urdf/xarm7/xarm7_robot_macro.xacro (robot description, xacro)
@@ -7,4 +7,5 @@
     velocity_control:=false
     add_gripper:=false
+    add_ft_sensor:=true
     add_bio_gripper:=false
     ros2_control_plugin:='uf_robot_hardware/UFRobotSystemHardware'
@@ -25,4 +26,8 @@
     <xacro:include filename="$(find xarm_description)/urdf/xarm7/xarm7.transmission.xacro" />
     <xacro:include filename="$(find xarm_description)/urdf/xarm7/xarm7.gazebo.xacro" />
+    <xacro:if value="${add_ft_sensor}">
+      <xacro:include filename="$(find xarm_description)/urdf/ft_sensor/ft_sensor.urdf.xacro"/>
+      <xacro:ft_sensor_urdf prefix="${prefix}" attach_to="${prefix}link7"/>
+    </xacro:if>
     <xacro:if value="${limited}">
       <xacro:if value="${is_ros2}">

File: xarm_description/urdf/xarm_device.urdf.xacro (robot description, xacro)
@@ -7,4 +7,5 @@
   <xacro:arg name="velocity_control" default="false"/>
   <xacro:arg name="add_gripper" default="false"/>
+  <xacro:arg name="add_ft_sensor" default="true"/>
   <xacro:arg name="add_vacuum_gripper" default="false"/>
   <xacro:arg name="add_bio_gripper" default="false"/>
@@ -39,4 +40,5 @@
   <xacro:arg name="mesh_suffix" default="stl"/>
   <xacro:arg name="kinematics_suffix" default=""/>
+  <xacro:include filename="$(find xarm_description)/urdf/ft_sensor/ft_sensor.urdf.xacro"/>
   <!-- load xarm device -->
   <xacro:include filename="$(find xarm_description)/urdf/xarm_device_macro.xacro" />
@@ -44,5 +46,5 @@
     effort_control="$(arg effort_control)" velocity_control="$(arg velocity_control)"
     add_gripper="$(arg add_gripper)" add_vacuum_gripper="$(arg add_vacuum_gripper)"
-    add_bio_gripper="$(arg add_bio_gripper)" dof="$(arg dof)"
+    add_bio_gripper="$(arg add_bio_gripper)" add_ft_sensor="$(arg add_ft_sensor)" dof="$(arg dof)"
     ros2_control_plugin="$(arg ros2_control_plugin)" robot_type="$(arg robot_type)"
     load_gazebo_plugin="true" ros2_control_params="$(arg ros2_control_params)"

File: xarm_description/urdf/xarm_device_macro.xacro (robot description, xacro)
@@ -8,4 +8,5 @@
     velocity_control:=false
     add_gripper:=false
+    add_ft_sensor:=true
     add_vacuum_gripper:=false
     add_bio_gripper:=false
@@ -43,4 +44,11 @@
     kinematics_suffix:=''
     ">
+    <!-- Add ft sensor -->
+    <xacro:if value="${add_ft_sensor}">
+      <xacro:property name="gripper_parent" value="${prefix}ft_sensor_link"/>
+    </xacro:if>
+    <xacro:unless value="${add_ft_sensor}">
+      <xacro:property name="gripper_parent" value="${prefix}link_eef"/>
+    </xacro:unless>
     <!-- Load Common Material -->
     <xacro:include filename="$(find xarm_description)/urdf/_private_macro.xacro" />
@@ -102,4 +110,5 @@
         ros2_control_plugin="${ros2_control_plugin}"
         add_gripper="${add_gripper}"
+        add_ft_sensor="${add_ft_sensor}"
         add_bio_gripper="${add_bio_gripper}"
         robot_ip="${robot_ip}"
@@ -120,4 +129,5 @@
           ros2_control_plugin="${ros2_control_plugin}"
           add_gripper="${add_gripper}"
+          add_ft_sensor="${add_ft_sensor}"
           add_bio_gripper="${add_bio_gripper}"
           robot_ip="${robot_ip}"
@@ -137,4 +147,5 @@
           ros2_control_plugin="${ros2_control_plugin}"
           add_gripper="${add_gripper}"
+          add_ft_sensor="${add_ft_sensor}"
           robot_ip="${robot_ip}"
           report_type="${report_type}"
@@ -153,4 +164,5 @@
           ros2_control_plugin="${ros2_control_plugin}"
           add_gripper="${add_gripper}"
+          add_ft_sensor="${add_ft_sensor}"
           add_bio_gripper="${add_bio_gripper}"
           robot_ip="${robot_ip}"
@@ -172,4 +184,5 @@
           ros2_control_plugin="${ros2_control_plugin}"
           add_gripper="${add_gripper}"
+          add_ft_sensor="${add_ft_sensor}"
           add_bio_gripper="${add_bio_gripper}"
           robot_ip="${robot_ip}"
@@ -189,4 +202,5 @@
           ros2_control_plugin="${ros2_control_plugin}"
           add_gripper="${add_gripper}"
+          add_ft_sensor="${add_ft_sensor}"
           add_bio_gripper="${add_bio_gripper}"
           robot_ip="${robot_ip}"
@@ -203,5 +217,5 @@
       <!-- Load RealSense D435i URDF -->
       <xacro:include filename="$(find xarm_description)/urdf/camera/realsense_d435i.urdf.xacro" />
-      <xacro:d435i_urdf prefix="${prefix}" add_d435i_links="${add_d435i_links}" />
+      <xacro:d435i_urdf prefix="${prefix}" add_d435i_links="${add_d435i_links}"/>
       <xacro:if value="${add_d435i_links}">
         <xacro:include filename="$(find xarm_description)/urdf/camera/realsense.gazebo.xacro" />
@@ -212,19 +226,28 @@
       <link name="${prefix}link_eef"/>
     </xacro:unless>
-    <joint name="${prefix}joint_eef" type="fixed">
-      <origin xyz="0 0 0" rpy="0 0 0" />
-      <parent link="${prefix}link${dof}" />
-      <child link="${prefix}link_eef" />
-    </joint>
+    <xacro:if value="${add_ft_sensor}">
+      <joint name="${prefix}joint_eef" type="fixed">
+        <origin xyz="0 0 0.029" rpy="0 0 0" />
+        <parent link="${prefix}ft_sensor_link" />
+        <child link="${prefix}link_eef" />
+      </joint>
+    </xacro:if>
+    <xacro:unless value="${add_ft_sensor}">
+      <joint name="${prefix}joint_eef" type="fixed">
+        <origin xyz="0 0 0.029" rpy="0 0 0" />
+        <parent link="${prefix}link${dof}" />
+      	<child link="${prefix}link_eef" />
+      </joint>
+    </xacro:unless>
     <xacro:if value="${add_gripper}">
       <xacro:if value="${robot_type == 'lite'}">
         <!-- Load Lite Gripper Model URDF -->
         <xacro:include filename="$(find xarm_description)/urdf/gripper/lite_gripper.urdf.xacro" />
-        <xacro:uflite_gripper_urdf prefix="${prefix}" attach_to="${prefix}link_eef" />
+        <xacro:uflite_gripper_urdf prefix="${prefix}" attach_to="${gripper_parent}" attach_xyz="0 0 0.029" />
       </xacro:if>
       <xacro:unless value="${robot_type == 'lite'}">
         <!-- Load XArm Gripper Model URDF -->
         <xacro:include filename="$(find xarm_description)/urdf/gripper/xarm_gripper_macro.xacro" />
-        <xacro:xarm_gripper_macro prefix="${prefix}" attach_to="${prefix}link_eef"
+        <xacro:xarm_gripper_macro prefix="${prefix}" attach_to="${gripper_parent}" attach_xyz="0 0 0.029"
           ros2_control_plugin="${ros2_control_plugin}" dof="${dof}" hard_interface="${hard_interface}" />
       </xacro:unless>
@@ -234,5 +257,5 @@
         <!-- Load BIO Gripper Model URDF -->
         <xacro:include filename="$(find xarm_description)/urdf/gripper/bio_gripper_macro.xacro" />
-        <xacro:bio_gripper_macro prefix="${prefix}" attach_to="${prefix}link_eef"
+        <xacro:bio_gripper_macro prefix="${prefix}" attach_to="${gripper_parent}" attach_xyz="0 0 0.029"
           ros2_control_plugin="${ros2_control_plugin}" dof="${dof}" hard_interface="${hard_interface}" />
       </xacro:unless>
@@ -242,10 +265,10 @@
         <!-- Load Lite Vacuum Gripper Model URDF -->
         <xacro:include filename="$(find xarm_description)/urdf/vacuum_gripper/lite_vacuum_gripper.urdf.xacro" />
-        <xacro:uflite_vacuum_gripper_urdf prefix="${prefix}" attach_to="${prefix}link_eef" />
+        <xacro:uflite_vacuum_gripper_urdf prefix="${prefix}" attach_to="${gripper_parent}" attach_xyz="0 0 0.029" />
       </xacro:if>
       <xacro:unless value="${robot_type == 'lite'}">
         <!-- Load XArm Vacuum Gripper Model URDF -->
         <xacro:include filename="$(find xarm_description)/urdf/vacuum_gripper/xarm_vacuum_gripper.urdf.xacro" />
-        <xacro:xarm_vacuum_gripper_urdf prefix="${prefix}" attach_to="${prefix}link_eef" />
+        <xacro:xarm_vacuum_gripper_urdf prefix="${prefix}" attach_to="${gripper_parent}" attach_xyz="0 0 0.029" />
       </xacro:unless>
     </xacro:if>

File: xarm_moveit_config/srdf/_xarm7_macro.srdf.xacro (robot description, xacro)
@@ -10,32 +10,9 @@
   <!-- SUBGROUPS: Groups can also be formed by referencing to already defined group names -->
   <xacro:macro name="xarm7_macro_srdf" params="prefix=''
-    add_gripper='false' add_vacuum_gripper='false' add_bio_gripper='false' add_other_geometry='false' ">
+    add_gripper='false' add_vacuum_gripper='false' add_bio_gripper='false' add_other_geometry='false'">
     <group name="${prefix}xarm7">
-      <joint name="${prefix}world_joint" />
-      <joint name="${prefix}joint1" />
-      <joint name="${prefix}joint2" />
-      <joint name="${prefix}joint3" />
-      <joint name="${prefix}joint4" />
-      <joint name="${prefix}joint5" />
-      <joint name="${prefix}joint6" />
-      <joint name="${prefix}joint7" />
-      <joint name="${prefix}joint_eef" />
-      <!-- To count in gripper TCP offset, if no need, please uncomment following 2 lines -->
-      <xacro:if value="${add_gripper}">
-        <joint name="${prefix}gripper_fix" />
-        <joint name="${prefix}joint_tcp" />
-      </xacro:if>
-      <xacro:if value="${not add_gripper and add_bio_gripper}">
-        <joint name="${prefix}bio_gripper_fix" />
-        <joint name="${prefix}joint_tcp" />
-      </xacro:if>
-      <xacro:if value="${not add_gripper and not add_bio_gripper and add_vacuum_gripper}">
-        <joint name="${prefix}vacuum_gripper_fix" />
-        <joint name="${prefix}joint_tcp" />
-      </xacro:if>
-      <xacro:if value="${not add_gripper and not add_bio_gripper and not add_vacuum_gripper and add_other_geometry}">
-        <joint name="${prefix}other_geometry_fix" />
-        <joint name="${prefix}joint_tcp" />
-      </xacro:if>
+       <chain
+         base_link="${prefix}link_base"
+         tip_link="${prefix}link_tcp"/>
     </group>
       <!-- GROUP STATES, Purpose, Define a named state for a particular group, in terms of joint values. This is useful to define states like 'folded arms' -->

File: xarm_moveit_config/srdf/xarm.srdf.xacro (robot description, xacro)
@@ -12,3 +12,9 @@
   <xacro:xarm_macro_srdf prefix="$(arg prefix)" dof="$(arg dof)" robot_type="$(arg robot_type)"
     add_gripper="$(arg add_gripper)" add_vacuum_gripper="$(arg add_vacuum_gripper)" add_bio_gripper="$(arg add_bio_gripper)" add_other_geometry="$(arg add_other_geometry)" />
+  <!-- allow links to overlap -->
+  <disable_collisions link1="link7" link2="ft_sensor_link" reason="adjacent_sensor"/>
+  <disable_collisions link1="link7" link2="link_eef" reason="adjacent_sensor"/>
+  <disable_collisions link1="link_eef" link2="ft_sensor_link" reason="adjacent_sensor"/>
+  <disable_collisions link1="link_eef" link2="link_eef" reason="adjacent_sensor"/>
+  <disable_collisions link1="xarm_gripper_base_link" link2="ft_sensor_link" reason="adjacent_sensor"/>
 </robot>
